File: PCB/tester serw.kicad_pcb (KiCad board)
At the start: 2 copper layers, 39.6 x 23.9 mm, 10 parts, among them CON1 AVR-ISP-10, IC1 ATTINY13A-SS, P1 servo, P2 servo, P3 servo, P4 power, SW1 button

Commit message: Add files via upload
Parts:
- RV1: footprint Potentiometers:Potentiometer_Alps-RK16-single -> Potentiometer_withoutlabel
Connections:
- CON1 pad 9: (no net) -> Net-(CON1-Pad9)
- IC1 pad 6: Net-(IC1-Pad6) -> Net-(CON1-Pad9)
- SW1 pad 2: Net-(IC1-Pad6) -> Net-(CON1-Pad9)
Routing:
- net Net-(CON1-Pad9): track 0.00 -> 26.2 mm, vias 0 -> 2
- net Net-(IC1-Pad6): track 19.3 -> 0.00 mm, vias 2 -> 0
Changed lines of the file:
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@@
-(kicad_pcb (version 4) (host pcbnew 4.0.4-stable)
+(kicad_pcb (version 4) (host pcbnew 4.0.7)
   (general
-    (links 28)
+    (links 29)
     (no_connects 0)
-    (area 115.824919 90.111 170.255001 116.280001)
+    (area 130.480999 92.253999 170.255001 116.280001)
     (thickness 1.6)
     (drawings 6)
-    (tracks 88)
+    (tracks 90)
     (zones 0)
     (modules 10)
@@
     (0 F.Cu signal)
     (31 B.Cu signal)
-    (32 B.Adhes user)
-    (33 F.Adhes user)
-    (34 B.Paste user)
-    (35 F.Paste user)
+    (32 B.Adhes user hide)
+    (33 F.Adhes user hide)
+    (34 B.Paste user hide)
+    (35 F.Paste user hide)
     (36 B.SilkS user)
     (37 F.SilkS user)
-    (38 B.Mask user)
-    (39 F.Mask user)
+    (38 B.Mask user hide)
+    (39 F.Mask user hide)
     (40 Dwgs.User user)
-    (41 Cmts.User user)
-    (42 Eco1.User user)
-    (43 Eco2.User user)
-    (44 Edge.Cuts user)
-    (45 Margin user)
-    (46 B.CrtYd user)
+    (41 Cmts.User user hide)
+    (42 Eco1.User user hide)
+    (43 Eco2.User user hide)
+    (44 Edge.Cuts user hide)
+    (45 Margin user hide)
+    (46 B.CrtYd user hide)
     (47 F.CrtYd user)
-    (48 B.Fab user)
-    (49 F.Fab user)
+    (48 B.Fab user hide)
+    (49 F.Fab user hide)
   )
   (setup
@@
     (pcbplotparams
       (layerselection 0x010f0_80000001)
-      (usegerberextensions false)
+      (usegerberextensions true)
       (excludeedgelayer true)
       (linewidth 0.100000)
@@
       (drillshape 0)
       (scaleselection 1)
-      (outputdirectory "D:/Projekty/kicad/tester serw/"))
+      (outputdirectory "D:/Projekty/kicad/tester serw/do produkcji"))
   )
   (net 0 "")
@@
   (net 5 "Net-(CON1-Pad7)")
   (net 6 "Net-(IC1-Pad3)")
-  (net 7 "Net-(IC1-Pad6)")
+  (net 7 "Net-(CON1-Pad9)")
   (net_class Default "To jest domyślna klasa połączeń."
     (clearance 0.3)
@@
     (add_net "Net-(CON1-Pad5)")
     (add_net "Net-(CON1-Pad7)")
+    (add_net "Net-(CON1-Pad9)")
     (add_net "Net-(IC1-Pad3)")
-    (add_net "Net-(IC1-Pad6)")
+  )
+  (module Potentiometer_withoutlabel (layer F.Cu)
+    (at 135.001 111.379 180)
+    (descr "Potentiometer, Alps, RK16, single, RevA, 30 July 2010,")
+    (tags "Potentiometer, Alps, RK16, single, RevA, 30 July 2010,")
+    (fp_text reference RV1 (at -3.599 16.379 180) (layer F.SilkS)
+      (effects (font (size 1 1) (thickness 0.15)))
+    )
+    (fp_text value 10K (at 0.127 16.002 180) (layer F.Fab)
+      (effects (font (size 1 1) (thickness 0.15)))
+    )
+    (fp_line (start 3.79984 -2.49936) (end 3.79984 -3.99796) (layer F.SilkS) (width 0.15))
+    (fp_line (start 3.79984 -3.99796) (end -6.70052 -3.99796) (layer F.SilkS) (width 0.15))
+    (fp_line (start -6.70052 -3.99796) (end -6.70052 -2.49936) (layer F.SilkS) (width 0.15))
+    (fp_line (start 3.79984 -2.49936) (end -6.70052 -2.49936) (layer F.SilkS) (width 0.15))
+    (fp_line (start -6.70052 -2.49936) (end -6.70052 12.50188) (layer F.SilkS) (width 0.15))
+    (fp_line (start -6.70052 12.50188) (end 3.79984 12.50188) (layer F.SilkS) (width 0.15))
+    (fp_line (start 3.79984 12.50188) (end 3.79984 -2.49936) (layer F.SilkS) (width 0.15))
+    (pad 2 thru_hole circle (at 0 5.00126 180) (size 2.49936 2.49936) (drill 1.19888) (layers *.Cu *.Mask F.SilkS)
+      (net 6 "Net-(IC1-Pad3)"))
+    (pad 3 thru_hole circle (at 0 10.00252 180) (size 2.49936 2.49936) (drill 1.19888) (layers *.Cu *.Mask F.SilkS)
+      (net 1 +BATT))
+    (pad 1 thru_hole circle (at 0 0 180) (size 2.49936 2.49936) (drill 1.19888) (layers *.Cu *.Mask F.SilkS)
+      (net 2 GND))
   )
   (module Capacitors_SMD:C_0805_HandSoldering (layer F.Cu)
@@
     (descr "10 pins through hole IDC header")
     (tags "IDC header socket VASCH")
-    (fp_text reference CON1 (at 5.08 -7.62) (layer F.SilkS)
+    (fp_text reference CON1 (at -0.009 -4.806) (layer F.SilkS)
       (effects (font (size 1 1) (thickness 0.15)))
     )
@@
     (pad 8 thru_hole oval (at 7.62 -2.54) (size 1.7272 1.7272) (drill 1.016) (layers *.Cu *.Mask)
       (net 2 GND))
-    (pad 9 thru_hole oval (at 10.16 0) (size 1.7272 1.7272) (drill 1.016) (layers *.Cu *.Mask))
+    (pad 9 thru_hole oval (at 10.16 0) (size 1.7272 1.7272) (drill 1.016) (layers *.Cu *.Mask)
+      (net 7 "Net-(CON1-Pad9)"))
     (pad 10 thru_hole oval (at 10.16 -2.54) (size 1.7272 1.7272) (drill 1.016) (layers *.Cu *.Mask)
       (net 2 GND))
@@
       (effects (font (size 1 1) (thickness 0.15)))
     )
-    (fp_text value servo (at 1.778 -8.763 90) (layer F.SilkS)
+    (fp_text value servo (at 1.778 -8.804 90) (layer F.SilkS)
       (effects (font (size 1 1) (thickness 0.15)))
     )
@@
       (effects (font (size 1 1) (thickness 0.15)))
     )
-    (fp_text value servo (at 7.493 -8.636 90) (layer F.SilkS)
+    (fp_text value servo (at 7.493 -8.804 90) (layer F.SilkS)
       (effects (font (size 1 1) (thickness 0.15)))
     )
@@
       (effects (font (size 1 1) (thickness 0.15)))
     )
-    (fp_text value servo (at -0.381 -8.763 90) (layer F.SilkS)
+    (fp_text value servo (at -0.381 -8.804 90) (layer F.SilkS)
       (effects (font (size 1 1) (thickness 0.15)))
     )
@@
       (net 3 "Net-(CON1-Pad1)"))
     (pad 6 smd rect (at 3.65 0.635) (size 1.7 0.65) (layers F.Cu F.Paste F.Mask)
-      (net 7 "Net-(IC1-Pad6)"))
+      (net 7 "Net-(CON1-Pad9)"))
     (pad 7 smd rect (at 3.65 -0.635) (size 1.7 0.65) (layers F.Cu F.Paste F.Mask)
       (net 5 "Net-(CON1-Pad7)"))
@@
       (rotate (xyz 0 0 0))
     )
-  )
-  (module Potentiometers:Potentiometer_Alps-RK16-single (layer F.Cu)
-    (at 135.001 111.379 180)
-    (descr "Potentiometer, Alps, RK16, single, RevA, 30 July 2010,")
-    (tags "Potentiometer, Alps, RK16, single, RevA, 30 July 2010,")
-    (fp_text reference RV1 (at -5.08 16.383 180) (layer F.SilkS)
-      (effects (font (size 1 1) (thickness 0.15)))
-    )
-    (fp_text value 10K (at 0.127 16.002 180) (layer F.Fab)
-      (effects (font (size 1 1) (thickness 0.15)))
-    )
-    (fp_line (start 0 14.00048) (end -6.70052 14.00048) (layer F.SilkS) (width 0.15))
-    (fp_line (start -6.70052 14.00048) (end -6.70052 12.40028) (layer F.SilkS) (width 0.15))
-    (fp_line (start 3.79984 -2.49936) (end 3.79984 -3.99796) (layer F.SilkS) (width 0.15))
-    (fp_line (start 3.79984 -3.99796) (end -6.70052 -3.99796) (layer F.SilkS) (width 0.15))
-    (fp_line (start -6.70052 -3.99796) (end -6.70052 -2.49936) (layer F.SilkS) (width 0.15))
-    (fp_line (start 3.79984 11.00074) (end 5.79882 11.00074) (layer F.SilkS) (width 0.15))
-    (fp_line (start 5.79882 11.00074) (end 5.79882 14.00048) (layer F.SilkS) (width 0.15))
-    (fp_line (start 5.79882 14.00048) (end 0 14.00048) (layer F.SilkS) (width 0.15))
-    (fp_line (start 0 14.00048) (end 0 12.50188) (layer F.SilkS) (width 0.15))
-    (fp_line (start 8.8011 2.00152) (end 18.80108 2.00152) (layer F.SilkS) (width 0.15))
-    (fp_line (start 18.80108 2.00152) (end 18.80108 8.001) (layer F.SilkS) (width 0.15))
-    (fp_line (start 18.80108 8.001) (end 8.8011 8.001) (layer F.SilkS) (width 0.15))
-    (fp_line (start 3.79984 1.50114) (end 8.8011 1.50114) (layer F.SilkS) (width 0.15))
-    (fp_line (start 8.8011 1.50114) (end 8.8011 8.50138) (layer F.SilkS) (width 0.15))
-    (fp_line (start 8.8011 8.50138) (end 3.79984 8.50138) (layer F.SilkS) (width 0.15))
-    (fp_line (start 3.79984 -2.49936) (end -6.70052 -2.49936) (layer F.SilkS) (width 0.15))
-    (fp_line (start -6.70052 -2.49936) (end -6.70052 12.50188) (layer F.SilkS) (width 0.15))
-    (fp_line (start -6.70052 12.50188) (end 3.79984 12.50188) (layer F.SilkS) (width 0.15))
-    (fp_line (start 3.79984 12.50188) (end 3.79984 -2.49936) (layer F.SilkS) (width 0.15))
-    (pad 2 thru_hole circle (at 0 5.00126 180) (size 2.49936 2.49936) (drill 1.19888) (layers *.Cu *.Mask F.SilkS)
-      (net 6 "Net-(IC1-Pad3)"))
-    (pad 3 thru_hole circle (at 0 10.00252 180) (size 2.49936 2.49936) (drill 1.19888) (layers *.Cu *.Mask F.SilkS)
-      (net 1 +BATT))
-    (pad 1 thru_hole circle (at 0 0 180) (size 2.49936 2.49936) (drill 1.19888) (layers *.Cu *.Mask F.SilkS)
-      (net 2 GND))
   )
   (module Buttons_Switches_SMD:SW_SPST_REED_CT05-XXXX-G1 (layer F.Cu)
@@
     (fp_line (start -3.25 -1.3) (end 3.25 -1.3) (layer F.SilkS) (width 0.12))
     (pad 2 smd rect (at 4.28 0) (size 2.5 2) (layers F.Cu F.Paste F.Mask)
-      (net 7 "Net-(IC1-Pad6)"))
+      (net 7 "Net-(CON1-Pad9)"))
     (pad 1 smd rect (at -4.28 0) (size 2.5 2) (layers F.Cu F.Paste F.Mask)
       (net 2 GND))
@@
   (segment (start 144.432 113.284) (end 141.90726 113.284) (width 0.8) (layer F.Cu) (net 6))
   (segment (start 141.90726 113.284) (end 135.001 106.37774) (width 0.8) (layer F.Cu) (net 6))
+  (segment (start 156.845 105.029) (end 158.369 103.505) (width 0.8) (layer F.Cu) (net 7))
+  (segment (start 158.369 103.505) (end 158.369 98.806) (width 0.8) (layer F.Cu) (net 7))
   (segment (start 156.845 105.029) (end 152.781 105.029) (width 0.8) (layer F.Cu) (net 7))
   (segment (start 152.781 105.029) (end 152.654 105.156) (width 0.8) (layer F.Cu) (net 7))
@@
     (polygon
       (pts
-        (xy 170.18 116.205) (xy 130.556 116.205) (xy 130.683 92.456) (xy 170.18 92.456)
+        (xy 130.6 92.4) (xy 170.2 92.4) (xy 170.2 116.2) (xy 130.6 116.2)
       )
     )
@@
     (polygon
       (pts
-        (xy 170.18 116.205) (xy 130.556 116.205) (xy 130.683 92.456) (xy 170.053 92.456)
+        (xy 130.6 92.4) (xy 170.2 92.4) (xy 170.2 116.2) (xy 130.6 116.2)
       )
     )
