File: PCB/tester serw.sch (KiCad schematic (older format))
At the start: 10 parts, among them CON1 AVR-ISP-10, IC1 ATTINY13A-SS, P1 servo, P2 servo, P3 servo, P4 power, SW1 button

Commit message: Add files via upload
Parts:
- RV1: symbol POT -> POT-RESCUE-tester_serw
Connections:
- net at IC1.6 (PB1(MISO/AIN1/OC0B/INT0/PCINT1)), SW1.2: now also CON1.9
Changed lines of the file:
@@
 EESchema Schematic File Version 2
+LIBS:tester serw-rescue
 LIBS:power
 LIBS:device
@@
 $EndComp
 $Comp
-L POT RV1
+L POT-RESCUE-tester_serw RV1
 U 1 1 598F3946
 P 3650 2970
@@
 	3950 3070 4110 3070
 Wire Wire Line
-	4705 2175 4010 2175
+	4010 2175 4705 2175
 Wire Wire Line
 	4010 2175 4010 2670
@@
 	4700 1775 4110 1775
 Connection ~ 3950 3070
+Connection ~ 4700 2175
 $EndSCHEMATC
